File: PCB/Devboard.kicad_pcb (KiCad board)
At the start: 2 copper layers, 21 x 51 mm, 37 parts, among them J1 USB_C_Receptacle_USB2.0_14P, J2 Conn_01x20, J3 Conn_01x20, J4 Conn_01x03, SW1 SW_Push, U1 RP2040, U2 NCP1117-3.3_SOT223, U3 W25Q16JVZPIQ TR, U4 BME680, Y1 12 MHz

Commit message: changed temperature sensor
Parts:
- removed U4: BME680, lcsc2:LGA-8_L3.0-W3.0-P0.80-TR
- added U5: BME280, Package_LGA:Bosch_LGA-8_2.5x2.5mm_P0.65mm_ClockwisePinNumbering, F.Cu at (163.6, 131.3)
Routing:
- net GND: track 68.4 -> 62.8 mm
- net TEMP_CSB: track 93.1 -> 90.8 mm
